File: Commodore Plus 4.kicad_pcb (KiCad board)
At the start: 2 copper layers, 284.7 x 158.9 mm, 236 parts, among them CN1 Conn_01x04, CN2 Conn_01x07, CN3 Conn_01x07, CN4 50PinEdge, CN5 Conn_01x08, CN6 Conn_01x08, CN7 Conn_01x08, CN8 Keyboard-Matrix, J1 Jumper_NC_Dual, J2 Jumper_NC_Dual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

Commit message: updates files for Kicad 8, some cleanup on libs and schematic
Other:
- net class Default removed
